Commit message: fixed bugs

File: robots/manipulator.URDF (robot description, URDF)
Before this commit: robot manipulator, 10 links, 9 joints
Links:
- link komodo_Arm_base_link: geometry collision mesh filename=package://manipulator_gazebo/robots/meshes_manipulator/komo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; visual mesh filename=package://manipulator_gazebo/robots/meshes_manipulator/komo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
- link komodo_base_rotation_link: geometry collision mesh filename=package://manipulator_gazebo/robots/meshes_manipulator/komo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; visual mesh filename=package://manipulator_gazebo/robots/meshes_manipulator/komo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
- link komodo_elbow1_link: geometry collision mesh filename=package://manipulator_gazebo/robots/meshes_manipulator/komo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; visual mesh filename=package://manipulator_gazebo/robots/meshes_manipulator/komo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
- link komodo_elbow2_link: geometry collision mesh filename=package://manipulator_gazebo/robots/meshes_manipulator/komo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; visual mesh filename=package://manipulator_gazebo/robots/meshes_manipulator/komo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
- link komodo_elevator_link: geometry collision mesh filename=package://manipulator_gazebo/robots/meshes_manipulator/komo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; visual mesh filename=package://manipulator_gazebo/robots/meshes_manipulator/komo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
- link komodo_left_finger_link: geometry collision mesh filename=package://manipulator_gazebo/robots/meshes_manipulator/komo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; visual mesh filename=package://manipulator_gazebo/robots/meshes_manipulator/komo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
- link komodo_right_finger_link: geometry collision mesh filename=package://manipulator_gazebo/robots/meshes_manipulator/komo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; visual mesh filename=package://manipulator_gazebo/robots/meshes_manipulator/komo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
- link komodo_shoulder_link: geometry collision mesh filename=package://manipulator_gazebo/robots/meshes_manipulator/komo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; visual mesh filename=package://manipulator_gazebo/robots/meshes_manipulator/komo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
- link komodo_wrist_link: geometry collision mesh filename=package://manipulator_gazebo/robots/meshes_manipulator/komo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; visual mesh filename=package://manipulator_gazebo/robots/meshes_manipulator/komo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

Commit message: added homework template

File: robots/manipulator.URDF (robot description, URDF)
Before this commit: robot manipulator, 10 links, 9 joints
Joints:
- joint komodo_elevator_joint: limit lower=0 upper=0.45 effort=500 velocity=0 -> lower=0 upper=0.45 effort=0 velocity=0
